Commit message: monopod model is mostly working and controlable. added ground plane from ignition-gym models repo and environment setup

File: monopod_v1/monopod_v1.urdf (robot description, URDF)
Before this commit: robot monopod_v1, 5 links, 4 joints
Links:
- removed link boom_Link
- removed link hip_Link
- removed link lower_leg_Link
- removed link upper_leg_Link
- added link boom_link, mass 0.12458; collision mesh filename=package://monopod_v1/meshes/boom_Link.STL; visual mesh filename=package://monopod_v1/meshes/boom_Link.STL
- added link hip_link, mass 0.2; collision mesh filename=package://monopod_v1/meshes/hip_Link.STL; visual mesh filename=package://monopod_v1/meshes/hip_Link.STL
- added link lower_leg_link, mass 0.054; collision mesh filename=package://monopod_v1/meshes/lower_leg_Link.STL; visual mesh filename=package://monopod_v1/meshes/lower_leg_Link.STL
- added link universal_link, mass 0.025
- added link upper_leg_link, mass 0.23078; collision mesh filename=package://monopod_v1/meshes/upper_leg_Link.STL; visual mesh filename=package://monopod_v1/meshes/upper_leg_Link.STL
- added link world
Joints:
- removed joint planarizer_joint
- added joint planarizer_01_joint: type continuous, parent base_link, child universal_link, origin xyz=0 0 0 rpy=0 0 0, axis 0 0 1
- added joint planarizer_02_joint: type continuous, parent universal_link, child boom_link, origin xyz=0 0 0 rpy=0 1.57 0, axis 0 1 0
- added joint world_to_base_link: type fixed, parent world, child base_link, origin xyz=0 0 0.075 rpy=0 3.14 0
- joint hip_joint: child hip_Link -> hip_link; origin xyz=0 0 1.4843 rpy=3.1416 0 1.3204 -> xyz=0 0 1.4843 rpy=3.1416 0 -1.57; parent boom_Link -> boom_link
- joint lower_leg_joint: child lower_leg_Link -> lower_leg_link; parent upper_leg_Link -> upper_leg_link
- joint upper_leg_joint: child upper_leg_Link -> upper_leg_link; parent hip_Link -> hip_link
