Commit message: fixed deafult positions of monopod in urdf. Monopod is now loaded by default in a vertical orientation. Positive position is rotating counter clockwise for both joints.

File: SIMP/monopod_v1/monopod_v1.urdf (robot description, URDF)
Before this commit: robot monopod_v1, 7 links, 6 joints
Joints:
- joint hip_joint: origin xyz=0 0 1.4843 rpy=3.1416 0 -1.57 -> xyz=0 0 1.4843 rpy=3.14159 0 -1.57
- joint lower_leg_joint: axis -1 0 0 -> 1 0 0; origin xyz=-0.041381 0 0.2 rpy=1.5622 0 0 -> xyz=0.03 0 0.2 rpy=0 0 0
- joint upper_leg_joint: axis -1 0 0 -> 1 0 0; origin xyz=-0.03 0.02 0 rpy=0.17161 -1.5708 -2.5959 -> xyz=-0.03 0.02 -0.115 rpy=-1.5708 1.5708 0
